File: lift/liftpcb/liftpcb.kicad_sch (KiCad schematic)
At the start: 1 part, among them U1 STM32C552CET6

Commit message: working on the layout
Parts:
- added C1: 0.01µF, symbol Device:C
- added C10: 0.1µF, symbol Device:C
- added C11: 1.5nF, symbol Device:C
- added C12, C14, C15: 100nF, symbol Device:C
- added C13: 100µF, symbol Device:C_Polarized_US
- added C16: 2.2µF, symbol Device:C
- added C17, C2, C8: 4.7µF, symbol Device:C
- added C3, C4, C5, C6, C7: 22µF, symbol Device:C
- added C9: 150pF, symbol Device:C
- added D1: SS34, Diode_SMD:D_SMA, symbol Device:D_Schottky
- added J1: Conn_01x02_Socket, Connector_AMASS:AMASS_XT30PW-F_1x02_P2.50mm_Horizontal, symbol Connector:Conn_01x02_Socket
- added J2: Conn_01x02_Socket, Connector_JST:JST_XH_B2B-XH-A_1x02_P2.50mm_Vertical, symbol Connector:Conn_01x02_Socket
- added L1: 15µH, symbol Device:L
- added R2: 5.9kΩ, symbol Device:R
- added R3: 549Ω, symbol Device:R
- added R5: 10kΩ, symbol Device:R
- added U2: TPS5430DDA, Package_SO:TI_SO-PowerPAD-8_ThermalVias, symbol Regulator_Switching:TPS5430DDA
- U1: footprint LQFP-48_STM -> Package_QFP:LQFP-48_7x7mm_P0.5mm
Connections:
- net at U1.22 (VCAP): now also C16.2
- net GND: now reaches U1.23 (VSS)
- net GND: now also U1.35 (VSS), U1.47 (VSS), U1.8 (VREF-), C10.2, C12.2, C13.2, C14.2, C15.2, C16.1, C17.2, C2.2, C3.2, C4.2, C5.2, C6.2, C7.2, C8.2, C9.2, D1.2 (A), J1.1 (Pin_1), R2.2, U2.6 (GND), U2.9 (GNDPAD)
- net +3.3V: now reaches U1.24 (VDD)
- net +3.3V: now also U1.36 (VDD), U1.48 (VDD), C11.2, C12.1, C14.1, C15.1, C17.1, C3.1, C4.1, C5.1, C6.1, C7.1, L1.2, R5.2
- new net: C1.2, D1.1 (K), L1.1, U2.8 (PH)
- new net: C11.1, C9.1, R2.1, R3.1, R5.1, U2.4 (VSENSE)
- new net: C1.1, U2.1 (BOOT)
- new net: C10.1, R3.2
- new net +24V: C13.1, C2.1, C8.1, J1.2 (Pin_2), U2.7 (VIN)
- new net CAN_H: J2.2 (Pin_2)
- new net CAN_L: J2.1 (Pin_1)
- no-connect marks 0 -> 1
Other:
- note added: "3.3V SUPPLY"
- moved on the sheet: U1A, U1B

Commit message: schematic updates
Parts:
- added C18, C19, C20: 100nF, symbol Device:C
- added C21, C22: 10pF, symbol Device:C
- added J3: Conn_01x05_Pin, Connector_PinHeader_2.54mm:PinHeader_1x05_P2.54mm_Vertical, symbol Connector:Conn_01x05_Pin
- added J4: Screw_Terminal_01x03, symbol Connector:Screw_Terminal_01x03
- added R1: 120Ω, Resistor_THT:R_Bare_Metal_Element_L12.4mm_W4.8mm_P11.40mm, symbol Device:R
- added SW1: SW_Push, Button_Switch_THT:SW_PUSH_6mm_H5mm, symbol Switch:SW_Push
- added U3: SN65HVD230DR, Package_SO:SOIC-8_3.9x4.9mm_P1.27mm, symbol Interface_CAN_LIN:SN65HVD230
- added Y1: 24 MHz, Crystal:Crystal_SMD_3225-4Pin_3.2x2.5mm, symbol Device:Crystal_GND24
Connections:
- net +3.3V: now also U1.9 (VREF+), C18.1, C19.1, J3.1 (Pin_1), U3.3 (VCC)
- net GND: now also C18.2, C19.2, C20.1, C21.1, C22.1, J3.5 (Pin_5), J4.1 (Pin_1), SW1.1, U3.2 (GND), U3.8 (Rs), Y1.2 (G), Y1.4 (G)
- net UART1_RX: now reaches U1.31 (PA10)
- net UART1_RX: now also J4.2 (Pin_2)
- net CAN_RX: now reaches U1.32 (PA11)
- net CAN_RX: now also U3.4 (R)
- net CAN_TX: now reaches U1.33 (PA12)
- net CAN_TX: now also U3.1 (D)
- net SWDIO: now reaches U1.34 (PA13)
- net SWDIO: now also J3.4 (Pin_4)
- net SWCLK: now reaches U1.37 (PA14)
- net SWCLK: now also J3.2 (Pin_2)
- net UART1_TX: now reaches U1.38 (PA15)
- net UART1_TX: now also J4.3 (Pin_3)
- net OSC_IN: now reaches U1.5 (PH0-OSC_IN)
- net OSC_IN: now also C21.2, Y1.1
- net OSC_OUT: now reaches U1.6 (PH1-OSC_OUT)
- net OSC_OUT: now also C22.2, Y1.3
- net NRST: now reaches U1.7 (NRST)
- net NRST: now also C20.2, J3.3 (Pin_3), SW1.2
- net CAN_H: no longer names the net of J2.2 (Pin_2)
- net CAN_H: now also R1.1, U3.7 (CANH)
- net CAN_L: no longer names the net of J2.1 (Pin_1)
- net CAN_L: now also R1.2, U3.6 (CANL)
- no-connect marks 1 -> 2
Other:
- note added: "CAN TX/RX"
- note added: "CRYSTAL"
- note added: "DEBUG HEADER"
- note added: "MC HEADER"
- note added: "PWR IN"
- note added: "STM32 PWR IN"
- company: (none) -> TERRIER RIDE ENGINEERING CLUB
- title: (none) -> LIFT DRIVE PCB
- moved on the sheet: C12, C14, C15, C16, C17, J1, J2, U1A, U1B

Commit message: leds
Parts:
- added D2, D3, D4, D5, D6: LED, symbol Device:LED
- added R4: 10kΩ, symbol Device:R
- J4: footprint (none) -> TerminalBlock_Phoenix:TerminalBlock_Phoenix_PT-1,5-3-5.0-H_1x03_P5.00mm_Horizontal
Connections:
- net +24V: now also D2.2 (A)
- net +3.3V: now also D3.2 (A)
- net GND: now also R4.2
- new net: D2.1 (K), R4.1
