File: lift/liftpcb/liftpcb.kicad_sch (KiCad schematic)
At the start: 43 parts, among them J1 Conn_01x02_Socket, J2 Conn_01x02_Socket, J3 Conn_01x05_Pin, J4 Screw_Terminal_01x03, SW1 SW_Push, U1 STM32C552CET6, U2 TPS5430DDA, U3 SN65HVD230DR, Y1 24 MHz

Commit message: leds and relays
Parts:
- removed D3: LED, symbol Device:LED
- removed J2: Conn_01x02_Socket, Connector_JST:JST_XH_B2B-XH-A_1x02_P2.50mm_Vertical, symbol Connector:Conn_01x02_Socket
- added D7, D8: 1N4148W, Diode_SMD:D_SOD-123, symbol Diode:1N4148W
- added J2: Conn_01x04_Socket, Connector_JST:JST_XH_S4B-XH-A_1x04_P2.50mm_Horizontal, symbol Connector:Conn_01x04_Socket
- added J5: Screw_Terminal_01x03, TerminalBlock_Phoenix:TerminalBlock_Phoenix_PT-1,5-3-5.0-H_1x03_P5.00mm_Horizontal, symbol Connector:Screw_Terminal_01x03
- added K1, K2: Relay_SPDT, symbol Relay:Relay_SPDT
- added Q1: MMBT3904, Package_TO_SOT_SMD:SOT-23, symbol Transistor_BJT:MMBT3904
- added R10: 10kΩ, Resistor_SMD:R_0603_1608Metric, symbol Device:R
- added R11: 100Ω, Resistor_SMD:R_0603_1608Metric, symbol Device:R
- added R12: 470Ω, Resistor_SMD:R_0603_1608Metric, symbol Device:R
- added R6: 13kΩ, symbol Device:R
- added R7, R9: 100kΩ, symbol Device:R
- added R8: 1kΩ, symbol Device:R
- D2: value LED -> GRN; footprint (none) -> LED_SMD:LED_0603_1608Metric
- D4: value LED -> YLW; footprint (none) -> LED_SMD:LED_0603_1608Metric
- D5: value LED -> WHT; footprint (none) -> LED_SMD:LED_0603_1608Metric
- D6: value LED -> RED; footprint (none) -> LED_SMD:LED_0603_1608Metric
- R4: footprint (none) -> Resistor_SMD:R_0603_1608Metric
Connections:
- net +24V: now also D8.1 (K), K1.11, K2.A2
- net GND: now also D7.2 (A), J5.2 (Pin_2), K1.A1, Q1.2 (E), R10.2, R11.2, R12.2, R6.2, R9.2
- net CAN_H: now reaches R1.1, U3.7 (CANH)
- net CAN_H: now also J2.4 (Pin_4)
- net CAN_L: now reaches R1.2, U3.6 (CANL)
- net CAN_L: now also J2.3 (Pin_3)
- net at D6.1 (K): now also R12.1
- net FAULT_LED: now reaches D6.2 (A)
- net FAULT_LED: now also U1.19 (PB1)
- net at D4.1 (K): now also R10.1
- net S+24V: now reaches D4.2 (A)
- net S+24V: now also J5.3 (Pin_3), K2.14, R7.1
- net at D5.1 (K): now also R11.1
- net COMM_LED: now reaches D5.2 (A)
- net COMM_LED: now also U1.18 (PB0)
- net S+24V_sense: now reaches U1.20 (PB2)
- net S+24V_sense: now also R6.1, R7.2
- new net: Q1.1 (B), R8.2, R9.1
- new net: K1.14, K2.11
- new net PWR_COIL: D8.2 (A), K2.A1, Q1.3 (C)
- new net PWR_CTL: R8.1
- new net SAFETY_COIL: D7.1 (K), J2.2 (Pin_2), K1.A2
Other:
- note added: "COMM"
- note added: "COMM ACTIVITY"
- note added: "FAULT"
- note added: "INDICATOR LIGHTS"
- note added: "LOGIC POWER"
- note added: "MC DATA"
- note added: "MC PWR"
- note added: "SAFETY COILS"
- note added: "SAFETY POWER"
- note removed: "MC HEADER"
- moved on the sheet: C20, D2, D4, D5, D6, J4, R4, SW1, U1A

Commit message: add fuse footprint
Parts:
- added F1: Fuse, trec:BLX-A, symbol Device:Fuse
Connections:
- net PWR_CTL is gone; now on net PWR_ENBL: R8.1
- net SAFETY_COIL: now also J2.1 (Pin_1); no longer J2.2 (Pin_2)
- net PWR_ENBL: now reaches U1.39 (PB3)
Other:
- moved on the sheet: D7, D8, K1, K2, Q1, R6, R7, R8, R9

Commit message: add enc
Parts:
- removed F1: Fuse, trec:BLX-A, symbol Device:Fuse
- added J6: Conn_01x06_Socket, Connector_JST:JST_PH_S6B-PH-K_1x06_P2.00mm_Horizontal, symbol Connector:Conn_01x06_Socket
- added R13, R14, R15, R16: 100Ω, symbol Device:R
Connections:
- net +3.3V: now also J6.1 (Pin_1)
- net GND: now also J6.6 (Pin_6)
- net at U1.10 (PA0): now also R13.2
- net at U1.11 (PA1): now also R14.2
- net at U1.12 (PA2): now also R15.2
- net at U1.29 (PA8): now also R16.2
- new net ENC_A: J6.3 (Pin_3), R13.1
- new net ENC_B: J6.4 (Pin_4), R14.1
- new net ENC_I: J6.5 (Pin_5), R15.1
- new net E_ABS: J6.2 (Pin_2), R16.1
Other:
- note added: "ENCODER"
- moved on the sheet: D7, D8, K1, K2, Q1, R6, R7, R8, R9

Commit message: add servo things
Parts:
- added C23: 470uF, symbol Device:C_Polarized_US
- added C24: 1µF, symbol Device:C
- added C25: 180µF, symbol Device:C_Polarized_US
- added D3: SS34, Diode_SMD:D_SMA, symbol Device:D_Schottky
- added J7: Screw_Terminal_01x03, TerminalBlock_Phoenix:TerminalBlock_Phoenix_PT-1,5-3-5.0-H_1x03_P5.00mm_Horizontal, symbol Connector:Screw_Terminal_01x03
- added L2: 68µH, symbol Device:L
- added U4: XL1509-5.0, Package_SO:SOIC-8_3.9x4.9mm_P1.27mm, symbol Regulator_Switching:XL1509-5.0
- J5: footprint TerminalBlock_Phoenix:TerminalBlock_Phoenix_PT-1,5-3-5.0-H_1x03_P5.00mm_Horizontal -> TerminalBlock_Phoenix:TerminalBlock_Phoenix_MKDS-1,5-2_1x02_P5.00mm_Horizontal; symbol Connector:Screw_Terminal_01x03 -> Connector:Screw_Terminal_01x02
Connections:
- net GND: now also J5.1 (Pin_1), C23.2, C24.2, C25.2, D3.2 (A), J7.1 (Pin_1), U4.4 (~{EN}), U4.5 (GND), U4.6 (GND), U4.7 (GND), U4.8 (GND); no longer J5.2 (Pin_2)
- net S+24V: now also J5.2 (Pin_2), C23.1, C24.1, U4.1 (VIN); no longer J5.3 (Pin_3)
- net SERVO_PWM: now reaches U1.16 (PA6)
- net SERVO_PWM: now also J7.2 (Pin_2)
- new net: D3.1 (K), L2.1, U4.2 (OUT)
- new net +5V: C25.1, J7.3 (Pin_3), L2.2, U4.3 (FB)
Other:
- note added: "5V SUPPLY"
- note added: "SERVO"
- moved on the sheet: J1, J2, J3, J4

Commit message: cleanup things
Connections:
- net GND: now also R6.1; no longer R6.2
- net S+24V: now also R7.2; no longer R7.1
- net S+24V_sense: now also R6.2, R7.1; no longer R6.1, R7.2
- no-connect marks 2 -> 4
Other:
- moved on the sheet: C12, C14, C15, C16, C17, C18, C20, C23, C24, C25, D2, D3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

Commit message: progres
Parts:
- added D10: WHT, LED_SMD:LED_0603_1608Metric, symbol Device:LED
- added D9: 1N4148W, Diode_SMD:D_SOD-123, symbol Diode:1N4148W
- added J8: Screw_Terminal_01x03, TerminalBlock_Phoenix:TerminalBlock_Phoenix_MKDS-1,5-2_1x02_P5.00mm_Horizontal, symbol Connector:Screw_Terminal_01x08
- added K3: Relay_SPDT, symbol Relay:Relay_SPDT
- added Q2, Q3, Q4, Q5, Q6: MMBT3904, Package_TO_SOT_SMD:SOT-23, symbol Transistor_BJT:MMBT3904
- added R17, R19, R21, R23, R25: 100kΩ, symbol Device:R
- added R18, R20, R22, R24, R26: 1kΩ, symbol Device:R
- added R27: 100Ω, Resistor_SMD:R_0603_1608Metric, symbol Device:R
- J5: symbol Connector:Screw_Terminal_01x02 -> Connector:Screw_Terminal_01x08
Connections:
- net GND: now also J5.4 (Pin_4), Q2.2 (E), Q3.2 (E), Q4.2 (E), Q5.2 (E), Q6.2 (E), R17.2, R19.2, R21.2, R23.2, R25.2, R27.2
- net S+24V: now also J5.8 (Pin_8), D9.1 (K), J8.2 (Pin_2), J8.4 (Pin_4), J8.6 (Pin_6), J8.8 (Pin_8), K3.A2; no longer J5.2 (Pin_2)
- net MOTOR_ENBL: now reaches U1.40 (PB4)
- net MOTOR_ENBL: now also R18.1
- new net: Q4.1 (B), R21.1, R22.2
- new net: Q2.1 (B), R17.1, R18.2
- new net: D10.1 (K), R27.1
- new net: Q3.1 (B), R19.1, R20.2
- new net: Q5.1 (B), R23.1, R24.2
- new net: Q6.1 (B), R25.1, R26.2
- new net M+: J5.6 (Pin_6), K3.11
- new net MC_M1A: J5.7 (Pin_7), K3.14
- new net MOTOR_COIL: D9.2 (A), K3.A1, Q2.3 (C)
- new net SOL1_DRAIN: J8.7 (Pin_7), Q3.3 (C)
- new net SOL1_GPIO: R20.1
- new net SOL2_DRAIN: J8.5 (Pin_5), Q4.3 (C)
- new net SOL2_GPIO: R22.1
- new net SOL3_DRAIN: J8.3 (Pin_3), Q5.3 (C)
- new net SOL3_GPIO: R24.1
- new net SOL4_DRAIN: J8.1 (Pin_1), Q6.3 (C)
- new net SOL4_GPIO: D10.2 (A), R26.1
- new net Shunt A: J5.5 (Pin_5), K3.12
- no-connect marks 4 -> 5
Other:
- note added: "SOLENOIDS"
- moved on the sheet: D7, D8, J1, J3, J6, J7, K1, K2, Q1, R6, R7, R8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
