File: lift/liftpcb/liftpcb.kicad_pcb (KiCad board)
At the start: 2 copper layers, 1 part, among them U1 STM32C552CET6

Commit message: working on the layout
Parts:
- added D1: SS34, Diode_SMD:D_SMA, F.Cu at (66.9, 175.9)
- added J1: Conn_01x02_Socket, Connector_AMASS:AMASS_XT30PW-F_1x02_P2.50mm_Horizontal, F.Cu at (52.7, 174.3)
- added J2: Conn_01x02_Socket, Connector_JST:JST_XH_B2B-XH-A_1x02_P2.50mm_Vertical, F.Cu at (66.3, 162.6)
- added U2: TPS5430DDA, Package_SO:TI_SO-PowerPAD-8_ThermalVias, F.Cu at (67.1, 170.4)
Connections:
- U1 pad 22: unconnected-(U1B-VCAP-Pad22) -> +3.3V
- U1 pad 23: unconnected-(U1B-VSS-Pad23) -> GND
- U1 pad 24: unconnected-(U1B-VDD-Pad24) -> +3.3V
- U1 pad 35: unconnected-(U1B-VSS-Pad35) -> GND
- U1 pad 36: unconnected-(U1B-VDD-Pad36) -> +3.3V
- U1 pad 47: unconnected-(U1B-VSS-Pad47) -> GND
- U1 pad 48: unconnected-(U1B-VDD-Pad48) -> +3.3V

Commit message: schematic updates
Parts:
- added J3: Conn_01x05_Pin, Connector_PinSocket_2.54mm:PinSocket_1x05_P2.54mm_Vertical, F.Cu at (115.0, 152.3)
- added R1: 120Ω, Resistor_THT:R_Bare_Metal_Element_L12.4mm_W4.8mm_P11.40mm, F.Cu at (115.0, 146.9)
- added SW1: SW_Push, Button_Switch_THT:SW_PUSH_6mm_H5mm, F.Cu at (119.3, 152.1)
- added U3: SN65HVD230DR, Package_SO:SOIC-8_3.9x4.9mm_P1.27mm, F.Cu at (121.5, 162.0)
- added Y1: 24 MHz, Crystal:Crystal_SMD_3225-4Pin_3.2x2.5mm, F.Cu at (128.4, 160.9)
- moved J2 37.0 mm to (30.6, 172.0)
- moved J1 5.51 mm to (47.8, 176.8)
Connections:
- J2 pad 1: CAN_L -> Net-(J2-Pin_1)
- J2 pad 2: CAN_H -> Net-(J2-Pin_2)
- U1 pad 22: +3.3V -> Net-(U1B-VCAP)
- U1 pad 31: unconnected-(U1A-PA10-Pad31) -> UART1_RX
- U1 pad 32: unconnected-(U1A-PA11-Pad32) -> CAN_RX
- U1 pad 33: unconnected-(U1A-PA12-Pad33) -> CAN_TX
- U1 pad 34: unconnected-(U1A-PA13-Pad34) -> SWDIO
- U1 pad 37: unconnected-(U1A-PA14-Pad37) -> SWCLK
- U1 pad 38: unconnected-(U1A-PA15-Pad38) -> UART1_TX
- U1 pad 5: unconnected-(U1A-PH0-OSC_IN-Pad5) -> OSC_IN
- U1 pad 6: unconnected-(U1A-PH1-OSC_OUT-Pad6) -> OSC_OUT
- U1 pad 7: unconnected-(U1A-NRST-Pad7) -> NRST
- U1 pad 8: unconnected-(U1B-VREF--Pad8) -> GND
- U1 pad 9: unconnected-(U1B-VREF+-Pad9) -> +3.3V

Commit message: add servo things
Parts:
- added D2: GRN, LED_SMD:LED_0603_1608Metric, F.Cu at (162.3, 106.6)
- added D4: YLW, LED_SMD:LED_0603_1608Metric, F.Cu at (162.3, 109.1)
- added D5: WHT, LED_SMD:LED_0603_1608Metric, F.Cu at (162.3, 111.7)
- added D6: RED, LED_SMD:LED_0603_1608Metric, F.Cu at (162.3, 114.3)
- added D7: 1N4148W, Diode_SMD:D_SOD-123, F.Cu at (171.2, 106.9)
- added D8: 1N4148W, Diode_SMD:D_SOD-123, F.Cu at (171.2, 110.3)
- added J2: Conn_01x04_Socket, Connector_JST:JST_XH_S4B-XH-A_1x04_P2.50mm_Horizontal, F.Cu at (118.7, 96.2)
- added J4: Screw_Terminal_01x03, TerminalBlock_Phoenix:TerminalBlock_Phoenix_PT-1,5-3-5.0-H_1x03_P5.00mm_Horizontal, F.Cu at (146.7, 96.7)
- added J5: Screw_Terminal_01x03, TerminalBlock_Phoenix:TerminalBlock_Phoenix_PT-1,5-3-5.0-H_1x03_P5.00mm_Horizontal, F.Cu at (146.7, 108.0)
- added J6: Conn_01x06_Socket, Connector_JST:JST_PH_S6B-PH-K_1x06_P2.00mm_Horizontal, F.Cu at (146.2, 116.7)
- added Q1: MMBT3904, Package_TO_SOT_SMD:SOT-23, F.Cu at (166.8, 117.5)
- added R10: 10kΩ, Resistor_SMD:R_0603_1608Metric, F.Cu at (166.3, 109.0)
- added R11: 100Ω, Resistor_SMD:R_0603_1608Metric, F.Cu at (166.3, 111.5)
- added R12: 470Ω, Resistor_SMD:R_0603_1608Metric, F.Cu at (166.3, 114.0)
- added R4: 10kΩ, Resistor_SMD:R_0603_1608Metric, F.Cu at (166.3, 106.5)
- J3: footprint Connector_PinSocket_2.54mm:PinSocket_1x05_P2.54mm_Vertical -> Connector_PinHeader_2.54mm:PinHeader_1x05_P2.54mm_Vertical
Connections:
- R1 pad 1: Net-(J2-Pin_2) -> CAN_H
- R1 pad 2: Net-(J2-Pin_1) -> CAN_L
- U1 pad 10: unconnected-(U1A-PA0-Pad10) -> Net-(U1A-PA0)
- U1 pad 11: unconnected-(U1A-PA1-Pad11) -> Net-(U1A-PA1)
- U1 pad 12: unconnected-(U1A-PA2-Pad12) -> Net-(U1A-PA2)
- U1 pad 18: unconnected-(U1A-PB0-Pad18) -> COMM_LED
- U1 pad 19: unconnected-(U1A-PB1-Pad19) -> FAULT_LED
- U1 pad 20: unconnected-(U1A-PB2-Pad20) -> S+24V_sense
- U1 pad 29: unconnected-(U1A-PA8-Pad29) -> Net-(U1A-PA8)
- U1 pad 39: unconnected-(U1A-PB3-Pad39) -> PWR_ENBL
- U3 pad 6: Net-(J2-Pin_1) -> CAN_L
- U3 pad 7: Net-(J2-Pin_2) -> CAN_H
