File: wiring diagram/wiring diagram.kicad_sch (KiCad schematic)
At the start: 5 parts, among them U2 RoboClaw Motor Controller, U3 5304 Gear Motor

Commit message: Update wiring diagram.kicad_sch
Changed lines of the file:
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@@
+	(wire
+		(pts
+			(xy 162.56 85.09) (xy 156.21 85.09)
+		)
+		(stroke
+			(width 0)
+			(type default)
+		)
+	)
 	(wire
 		(pts
@@
 	(wire
 		(pts
+			(xy 163.83 78.74) (xy 91.44 78.74)
+		)
+		(stroke
+			(width 0)
+			(type default)
+		)
+	)
+	(wire
+		(pts
 			(xy 91.44 96.52) (xy 91.44 92.71)
 		)
@@
 	(wire
 		(pts
+			(xy 163.83 87.63) (xy 163.83 78.74)
+		)
+		(stroke
+			(width 0)
+			(type default)
+		)
+	)
+	(wire
+		(pts
 			(xy 91.44 88.9) (xy 95.25 88.9)
 		)
@@
 	(wire
 		(pts
-			(xy 156.21 85.09) (xy 156.21 78.74)
-		)
-		(stroke
-			(width 0)
-			(type default)
-		)
-	)
-	(wire
-		(pts
 			(xy 158.75 110.49) (xy 154.94 110.49)
 		)
@@
 	(wire
 		(pts
-			(xy 91.44 76.2) (xy 163.83 76.2)
-		)
-		(stroke
-			(width 0)
-			(type default)
-		)
-	)
-	(wire
-		(pts
 			(xy 154.94 107.95) (xy 161.29 107.95)
 		)
@@
 	(wire
 		(pts
-			(xy 163.83 76.2) (xy 163.83 87.63)
-		)
-		(stroke
-			(width 0)
-			(type default)
-		)
-	)
-	(wire
-		(pts
 			(xy 161.29 107.95) (xy 161.29 135.89)
 		)
@@
 	(wire
 		(pts
-			(xy 156.21 78.74) (xy 91.44 78.74)
-		)
-		(stroke
-			(width 0)
-			(type default)
-		)
-	)
-	(wire
-		(pts
 			(xy 124.46 132.08) (xy 157.48 132.08)
 		)
@@
 		)
 		(stroke
+			(width 0)
+			(type default)
+		)
+	)
+	(wire
+		(pts
+			(xy 91.44 76.2) (xy 162.56 76.2)
+		)
+		(stroke
+			(width 0)
+			(type default)
+		)
+	)
+	(wire
+		(pts
+			(xy 162.56 76.2) (xy 162.56 85.09)
+		)
+		(stroke
